File: COMMS_BOARD.kicad_sch (KiCad schematic)
At the start: 20 parts, among them U3 ESP32-WROOM-32E

Commit message: 66
Other:
- note added: "on actual build: VTX EN: GPIO 5 cutteR: GPIO4"
- note removed: "UARTS are flipped here"
Changed lines of the file:
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@@
 		)
 	)
-	(text "UARTS are flipped here"
+	(text "220ohm @100MHz\n"
 		(exclude_from_sim no)
-		(at 98.552 80.518 0)
+		(at 134.366 165.862 0)
 		(effects
 			(font
@@
 		)
 	)
-	(text "220ohm @100MHz\n"
+	(text "on actual build: VTX EN: GPIO 5\ncutteR: GPIO4\n"
 		(exclude_from_sim no)
-		(at 134.366 165.862 0)
+		(at 94.996 26.924 0)
 		(effects
 			(font
@@
 			"AAAAAAAAAAAAAAAAAAAAAAAAAAAAAAAAAAAAAAAAAAAAAAAAAAAAAAAAAAAAAAAAAAAAAAAAAAAA"
 			"AAAAAAAAAAAAAAAAAAAAAAAAAAAAAAAAAAAAAAAAAAAAAAAAAAAAAAAAAAAAAAAAAAAAAAAAAAAA"
+			"AAAAAAAAAAAAAAAAAAAAAAAAAAAAAAAAAAAAAAAAAAAAAAAAAAAAAAAAAAAAAAAAAAAAAAAAAAAA"
+			"AAAAAAAAAAAAAAAAAAAAAAAAAAAAAAAAAAAAAAAAAAAAAAAAAAAAAAAAAAAAAAAAAAAAAAAAAAAA"
+			"AAAAAAAAAAAAAAAAAAAAAAAAAAAAAAAAAAAAAAAAAAAAAAAAAAAAAAAAAAAAAAAAAAAAAAAAAAAA"
+			"AAAAAAAAAAAAAAAAAAAAAAAAAAAAAAAAAAAAAAAAAAAAAAAAAAAAAAAAAAAAAAAAAAAAAAAAAAAA"
+			"AAAAAAAAAAAAAAAAAAAAAAAAAAAAAAAAAAAAAAAAAAAAAAAAAAAAAAAAAAAAAAAAAAAAAAAAAAAA"
+			"AAAAAAAAAAAAAAAAAAAAAAAAAAAAAAAAAAAAAAAAAAAAAAAAAAAAAAAAAAAAAAAAAAAAAAAAAAAA"
+			"AAAAAAAAAAAAAAAAAAAAAAAAAAAAAAAAAAAAAAAAAAAAAAAAAAAAAAAAAAAAAAAAAAAAAAAAAAAA"
+			"AAAAAAAAAAAAAAAAAAAAAAAAAAAAAAAAAAAAAAAAAAAAAAAAAAAAAAAAAAAAAAAAAAAAAAAAAAAA"
+			"AAAAAAAAAAAAAAAAAAAAAAAAAAAAAAAAAAAAAAAAAAAAAAAAAAAAAAAAAAAAAAAAAAAAAAAAAAAA"
+			"AAAAAAAAAAAAAAAAAAAAAAAAAAAAAAAAAAAAAAAAAAAAAAAAAAAAAAAAAAAAAAAAAAAAAAAAAAAA"
+			"AAAAAAAAAAAAAAAAAAAAAAAAAAAAAAAAAAAAAAAAAAAAAAAAAAAAAAAAAAAAAAAAAAAAAAAAAAAA"
+			"AAAAAAAAAAAAAAAAAAAAAAAAAAAAAAAAAAAAAAAAAAAAAAAAAAAAAAAAAAAAAAAAAAAAAAAAAAAA"
+			"AAAAAAAAAAAAAAAAAAAAAAAAAAAAAAAAAAAAAAAAAAAAAAAAAAAAAAAAAAAAAAAAAAAAAAAAAAAA"
+			"AAAAAAAAAAAAAAAAAAAAAAAAAAAAAAAAAAAAAAAAAAAAAAAAAAAAAAAAAAAAAAAAAAAAAAAAAAAA"
+			"AAAAAAAAAAAAAAAAAAAAAAAAAAAAAAAAAAAAAAAAAAAAAAAAAAAAAAAAAAAAAAAAAAAAAAAAAAAA"
+			"AAAAAAAAAAAAAAAAAAAAAAAAAAAAAAAAAAAAAAAAAAAAAAAAAAAAAAAAAAAAAAAAAAAAAAAAAAAA"
+			"AAAAAAAAAAAAAAAAAAAAAAAAAAAAAAAAAAAAAAAAAAAAAAAAAAAAAAAAAAAAAAAAAAAAAAAAAAAA"
+			"AAAAAAAAAAAAAAAAAAAAAAAAAAAAAAAAAAAAAAAAAAAAAAAAAAAAAAAAAAAAAAAAAAAAAAAAAAAA"
 			"AAAAAAAAAAAAAAAAAAAAAAAAAAAAAAAAAAAAAA=="
 		)
@@
 			"////////////////////////////////////////////////////////////////////////////"
 			"////////////////////////////////////////////////////////////////////////////"
-			"/////////////////////////////////////////////w=="
-		)
-	)
+			"/////////////////////////////////////////////zNFZGM3NitZd3k0TGdvSytBZTRyeHdQ"
+			"VlBPTE05OXFMTGxlMzZQYnJqaGhwRHVWVDBVNlBwU0djcmc2cHlZMm1JVFoweE9rSW1qc3Q5NDQ0"
+			"M0RDQnh5eUNGUllXSkVhT0I0MnFiaUhqRmlSSExvb1ljbUF3Y09qRWljVEp3YWFqVWVhdHhrdXFa"
+			"T25ScVNnYUFCUmVQSGp3OHBta1FqZ3RnUHBFYnVpaXV1Q0UyYk5pMms1YWRNbVJKU1kxbkt4TkVn"
+			"SVJvU0dnSWF3b2tUSjRaNXUrQ0NDMkxiOUF2ay96UllORkEwUHFRM01abnNLNGFJU0FGR2lnYVQ4"
+			"dUdZMlErTytaeHp6Z216aEJHZy9DZzNEQmxSRHRhSjZjQmMwZkFRRGFHeHBKRmlmMmk0aVFxeVBn"
+			"d2EyMVVFUmczOGhBa1RRcXdicVUrYW9xSnFERTgrK2VRUWtWUEUvaUQyRDJYTFZzdHo3SWhyQUpV"
+			"eWNlM2F0UXZKdkdtL0tGZWtVYk1jSXdZRUE0eG8wRlVHR0F2T0NkY0lKb0JyVWlhT2hweGxPQmZz"
+			"SjJhSTgwVVpjMjN4ZjhvZU04S0RCdHZpZXNac2NCejhEZlF0Sk1xRkdlRmF4OVJnOXRnbitoS3k3"
+			"NXhiekJqbkVjT3BNaEl5UzVnanBLaVJ5bGJYdS9wMlhuamhoU0hkRDFyK2hCTk9DT25oaEljanhM"
+			"RWc5ZzNwM01ra2FzQ09sdFAzdXY2NU41SHVFOHBJNWNYOXpQVkZlV0N5dUtlNW50aGZyZ2V1Uzhx"
+			"ZjZ4d2pSMWxpdGpGWW5LOEJBd2JFUHJOOW1Va2RHK2NNWXpadjNyeTROcmt2ZUFqaTJ1WWNzeDRl"
+			"VERnbXRzVTF6bm1WK2VJZTQwRUo2YUZFWmFON1hHV3JNbFcwa25Wb1BhWjIyTVFaa3hOazRqQVJO"
+			"TWFEQncrT2lNem8wYU9Udm4zN2hsa2l4VUlGVG9UdXNNTU9pNG9Za3lRVEorTXdhTkNna0tJNmFu"
+			"VDIyR09QRUEwMW9vRkZ1KzY2YTBoL3E2SmVmLzMxUTNvYXB3RkJNZ2FLUmltRlNJT0RTcGs0cFpG"
+			"WXBuUG56dEdIalBReGpRUVJRUnBZb2s5SEhYVlVOR1kwK0pRUDVtYnp6VGVQdENITHN3ODBXRFIy"
+			"bEFXLzJXdXZ2V0k5R0RaTURJMFpuOU9vcXFHam9ULzQ0SU9qTWNNY1lGNklMckZkK3BYUjBOS3dz"
+			"djZkZDk0NWZvZng0TGN5RGoxNzlnd1JUVUlISFhSUWFKZGRkZ2twUmEzSW5JdzE1aFR0czg4K0la"
+			"V055a29STzdhRjl0OS8vMUFwRTZkcmdPc0ZhVUFFSmgvcA=="
+		)
+	)
