File: COMMS_BOARD.kicad_sch (KiCad schematic)
At the start: 20 parts, among them U3 ESP32-WROOM-32E

Commit message: ADDE IMU
Connections:
- net CUTTER_EN renamed INT1_ACCEL
- net VTX_EN renamed INT1_GYRO

Commit message: EE
Other:
- note added: "IO34 AND 35 are inputs, so these are interrupts from IMU"
Changed lines of the file:
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@@
+		)
+	)
+	(text "IO34 AND 35 are inputs, so these are interrupts from IMU"
+		(exclude_from_sim no)
+		(at 88.9 120.904 0)
+		(effects
+			(font
+				(size 1.27 1.27)
+			)
 		)
 	)
