File: COMMS_BOARD_EXTERNAL_CONNS.kicad_sch (KiCad schematic)
At the start: 12 parts, among them J2 Conn_01x02, J3 Conn_01x04, J7 Conn_01x06, J8 Conn_01x04, U5 USBLC6-2SC6

Commit message: ADDE IMU
Parts:
- removed D3, D8: PESD3V3Z1BCSFYL, SamacSys_Parts:PMEG3005AESFYL, symbol Samac_sys:PESD3V3Z1BCSFYL
- removed J7: Conn_01x06, Connector_JST:JST_PH_B6B-PH-K_1x06_P2.00mm_Vertical, symbol Connector_Generic:Conn_01x06
- added J7: Conn_01x04, Connector_JST:JST_PH_S4B-PH-K_1x04_P2.00mm_Horizontal, symbol Connector_Generic:Conn_01x04
Connections:
- net +3V3: now also J7.1 (Pin_1)
- net GND: now also J7.4 (Pin_4)
- net I2C2_SDA: now also J7.3 (Pin_3)
- net I2C2_SDL: now also J7.2 (Pin_2)

Commit message: REV2 RELEASE
IO34 AND 35 are inputs, so these are interrupts from IMU
Parts:
- J2: footprint Connector_JST:JST_XH_B2B-XH-A_1x02_P2.50mm_Vertical -> Connector_JST:JST_XH_S2B-XH-A-1_1x02_P2.50mm_Horizontal
Changed lines of the file:
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@@
 			)
 		)
-		(property "Footprint" "Connector_JST:JST_XH_B2B-XH-A_1x02_P2.50mm_Vertical"
+		(property "Footprint" "Connector_JST:JST_XH_S2B-XH-A-1_1x02_P2.50mm_Horizontal"
 			(at 49.53 142.24 0)
 			(hide yes)
